File: custom_pcb/smartlada_revA/smartlada_revA.kicad_sch (KiCad schematic)
At the start: 30 parts, among them J1 +12V IN, J2 LAMPS_OUT, J3 DEVBOARD PINS, Q1 AOD4184A, Q2 AOD4184A, Q3 AOD4184A, Q4 AOD4184A, Q5 AOD4185, U1 TPS54202DDC

Commit message: Add Rev B/Rev C boards + firmware; repo hygiene
PCB: Rev C (product) routed/verified/gerbers/mechanical, ordered; Rev B
(learning 4-layer) + docs; Rev A updates; Vendor lib new footprints
(Faston TE_1217754-1, WS2812B, ESP32-C6-WROOM-1-N16, USB-B, tactile) + 3D shapes.

Firmware: SmartLadaRevC (fork of RevB with Rev C pin remap, builds;
PD-gating pending -> CODE_HANDOFF.md); SmartLadaRevB (modular UI, effects, fonts).

Docs/tooling: Rev C verification/procurement/handoffs, fab READMEs, KiCad
workflow, test sketches, tools; UI fonts limited to chosen orp/dweep.

Repo hygiene: .gitignore excludes timelapse video, payment docs, backups,
datasheets, renders, node_modules, unused font experiments.

Co-Authored-By: Claude Opus 4.8 <noreply@anthropic.com>
Parts:
- C1: MPN (none) -> EEUFR1E101; Manufacturer (none) -> Panasonic
- C2: MPN (none) -> GRM21BR71E104KA01L; Manufacturer (none) -> Murata
- C3, C4: MPN (none) -> HLC1210X7R106K500N; Manufacturer (none) -> Walsin
- C5: MPN (none) -> GRM188R72A104KA35D; Manufacturer (none) -> Murata
- C6, C7: MPN (none) -> GRT21BR61E226ME13L; Manufacturer (none) -> Murata
- D1: MPN (none) -> SS14-E3/61T; Manufacturer (none) -> Vishay
- F1: MPN (none) -> S1052-1; MPN_Fuse (none) -> FS-52GT-4.0/250; Manufacturer (none) -> RUICHI
- J1: MPN (none) -> DG127-5.0-02P-14-00Z(H); Manufacturer (none) -> Degson
- J2: footprint TerminalBlock:TerminalBlock_MaiXu_MX126-5.0-05P_1x05_P5.00mm -> TerminalBlock_Phoenix:TerminalBlock_Phoenix_MPT-0,5-5-2.54_1x05_P2.54mm_Horizontal; MPN (none) -> DG308-2.54-05P-14-00ZH; Manufacturer (none) -> Degson
- J3: MPN (none) -> PLS-40 (alt L-KLS1-207-1-40-S); Manufacturer (none) -> KLS
- L1: MPN (none) -> CDRH6D28NP-100NC; Manufacturer (none) -> Sumida
- Q1, Q2, Q3, Q4: MPN (none) -> AOD4184A; Manufacturer (none) -> Alpha & Omega (AOS)
- Q5: MPN (none) -> AOD4185; Manufacturer (none) -> Alpha & Omega (AOS)
- R1, R2, Rpd1, Rpd2, Rpd3, Rpd4: MPN (none) -> ERJP06F1003V; Manufacturer (none) -> Panasonic
- R3: MPN (none) -> RC0805FR-0713K7L; Manufacturer (none) -> Yageo
- Rg1, Rg2, Rg3, Rg4: MPN (none) -> RT0805BRD07100RL; Manufacturer (none) -> Yageo
- U1: MPN (none) -> TPS54202DDCR; Manufacturer (none) -> Texas Instruments
